Commit message: structure is updated

File: my_robot/urdf/my_robot.xacro (robot description, xacro)
@@ -3,9 +3,4 @@
   <xacro:include filename="$(find my_robot)/urdf/my_robot.gazebo" />
   <link name="robot_footprint"></link>
-  <joint name="robot_footprint_joint" type="fixed">
-  <origin xyz="0 0 0" rpy="0 0 0" />
-  <parent link="robot_footprint"/>
-  <child link="chassis" />
-  </joint>
   <link name='chassis'>
     <pose>0 0 0.1 0 0 0</pose>
@@ -16,6 +11,5 @@
           ixx="0.1" ixy="0" ixz="0"
           iyy="0.1" iyz="0"
-          izz="0.1"
-      />
+          izz="0.1"/>
     </inertial>
     <collision name='collision'>
@@ -56,13 +50,17 @@
     </visual>
   </link>
+  <joint name="robot_footprint_joint" type="fixed">
+    <origin xyz="0 0 0" rpy="0 0 0" />
+    <parent link="robot_footprint"/>
+    <child link="chassis" />
+  </joint>
   <link name='left_wheel'>
     <inertial>
-    <origin xyz="0 0 0" rpy="0 1.5707 1.5707"/>
-    <mass value="5"/>
-      <inertia
-          ixx="0.1" ixy="0" ixz="0"
-          iyy="0.1" iyz="0"
-          izz="0.1"
-      />
+      <origin xyz="0 0 0" rpy="0 1.5707 1.5707"/>
+      <mass value="5"/>
+        <inertia
+            ixx="0.1" ixy="0" ixz="0"
+            iyy="0.1" iyz="0"
+            izz="0.1" />
     </inertial>
     <visual>
@@ -80,20 +78,19 @@
   </link>
   <joint name="left_wheel_hinge" type="continuous">
-  <origin xyz="0 0.15 0" rpy="0 0 0" />
-  <parent link="chassis"/>
-  <child link="left_wheel" />
-  <axis xyz="0 1 0" rpy="0 0 0"/>
-  <limit effort="10000" velocity="1000"/>
-  <dynamics damping="1.0" friction="1.0"/>
+    <origin xyz="0 0.15 0" rpy="0 0 0" />
+    <parent link="chassis"/>
+    <child link="left_wheel" />
+    <axis xyz="0 1 0" rpy="0 0 0"/>
+    <limit effort="10000" velocity="1000"/>
+    <dynamics damping="1.0" friction="1.0"/>
   </joint>
   <link name='right_wheel'>
     <inertial>
-    <origin xyz="0 -0.3 0" rpy="0 1.5707 1.5707"/>
-    <mass value="5"/>
+      <origin xyz="0 -0.3 0" rpy="0 1.5707 1.5707"/>
+      <mass value="5"/>
       <inertia
           ixx="0.1" ixy="0" ixz="0"
           iyy="0.1" iyz="0"
-          izz="0.1"
-      />
+          izz="0.1"/>
     </inertial>
     <visual>
@@ -111,72 +108,72 @@
   </link>
   <joint name="right_wheel_hinge" type="continuous">
-  <origin xyz="0 0.15 0" rpy="0 0 0" />
-  <parent link="chassis"/>
-  <child link="right_wheel" />
-  <axis xyz="0 1 0" rpy="0 0 0"/>
-  <limit effort="10000" velocity="1000"/>
-  <dynamics damping="1.0" friction="1.0"/>
+    <origin xyz="0 0.15 0" rpy="0 0 0" />
+    <parent link="chassis"/>
+    <child link="right_wheel" />
+    <axis xyz="0 1 0" rpy="0 0 0"/>
+    <limit effort="10000" velocity="1000"/>
+    <dynamics damping="1.0" friction="1.0"/>
   </joint>
-<link name="camera">
-<inertial>
-  <origin xyz="0 0 0" rpy="0 0 0"/>
-  <mass value="0.1"/>
-  <inertia ixx="1e-6" ixy="0" ixz="0.0" iyy="1e-6" iyz="0" izz="1e-6"/>
-</inertial>
-<collision>
-  <origin xyz="0 0 0" rpy="0 0 0"/>
-  <geometry>
-    <box size="0.05 0.05 0.05"/>
-  </geometry>
-</collision>
-<visual>
-  <origin xyz="0 0 0" rpy="0 0 0"/>
-  <geometry>
-    <box size="0.05 0.05 0.05"/>
-  </geometry>
-</visual>
-</link>
-<joint name="camera_joint" type="fixed">
-  <origin xyz="0.2 0.0 0.0" rpy="0.0 0.0 0.0"/>
-  <parent link="chassis"/>
-  <child link="camera"/>
-  <axis xyz="0.0 1.0 0.0"/>
-</joint>
-<link name="hokuyo">
-<inertial>
-  <origin xyz="0 0 0" rpy="0 0 0"/>
-  <mass value="1e-5"/>
-  <inertia ixx="1e-6" ixy="0" ixz="0" iyy="1e-6" iyz="0" izz="1e-6"/>
-</inertial>
-<collision>
-  <origin xyz="0 0 0" rpy="0 0 0"/>
-  <geometry>
-    <box size="0.1 0.1 0.1"/>
-  </geometry>
-</collision>
-<visual>
-  <origin xyz="0 0 0" rpy="0 0 0"/>
-  <geometry>
-    <mesh filename="package://my_robot/meshes/hokuyo.dae"/>
-  </geometry>
-</visual>
-</link>
-<joint name="hokuyo_joint" type="fixed">
-  <origin xyz="0.15 0.0 0.1" rpy="0.0 0.0 0.0"/>
-  <parent link="chassis"/>
-  <child link="hokuyo"/>
-  <axis xyz="0.0 1.0 0.0"/>
-</joint>
-<gazebo reference="chassis">
-  <material>Gazebo/Yellow</material>
-</gazebo>
-<gazebo reference="left_wheel">
-  <material>Gazebo/Yellow</material>
-</gazebo>
-<gazebo reference="right_wheel">
-  <material>Gazebo/Yellow</material>
-</gazebo>
-<gazebo reference="camera">
-  <material>Gazebo/Yellow</material>
-</gazebo>
+  <link name="camera">
+    <inertial>
+      <origin xyz="0 0 0" rpy="0 0 0"/>
+      <mass value="0.1"/>
+      <inertia ixx="1e-6" ixy="0" ixz="0.0" iyy="1e-6" iyz="0" izz="1e-6"/>
+    </inertial>
+    <collision>
+      <origin xyz="0 0 0" rpy="0 0 0"/>
+      <geometry>
+        <box size="0.05 0.05 0.05"/>
+      </geometry>
+    </collision>
+    <visual>
+      <origin xyz="0 0 0" rpy="0 0 0"/>
+      <geometry>
+        <box size="0.05 0.05 0.05"/>
+      </geometry>
+    </visual>
+  </link>
+  <joint name="camera_joint" type="fixed">
+    <origin xyz="0.2 0.0 0.0" rpy="0.0 0.0 0.0"/>
+    <parent link="chassis"/>
+    <child link="camera"/>
+    <axis xyz="0.0 1.0 0.0"/>
+  </joint>
+  <link name="hokuyo">
+    <inertial>
+      <origin xyz="0 0 0" rpy="0 0 0"/>
+      <mass value="1e-5"/>
+      <inertia ixx="1e-6" ixy="0" ixz="0" iyy="1e-6" iyz="0" izz="1e-6"/>
+    </inertial>
+    <collision>
+      <origin xyz="0 0 0" rpy="0 0 0"/>
+      <geometry>
+        <box size="0.1 0.1 0.1"/>
+      </geometry>
+    </collision>
+    <visual>
+      <origin xyz="0 0 0" rpy="0 0 0"/>
+      <geometry>
+        <mesh filename="package://my_robot/meshes/hokuyo.dae"/>
+      </geometry>
+    </visual>
+  </link>
+  <joint name="hokuyo_joint" type="fixed">
+    <origin xyz="0.15 0.0 0.1" rpy="0.0 0.0 0.0"/>
+    <parent link="chassis"/>
+    <child link="hokuyo"/>
+    <axis xyz="0.0 1.0 0.0"/>
+  </joint>
+  <gazebo reference="chassis">
+    <material>Gazebo/Yellow</material>
+  </gazebo>
+  <gazebo reference="left_wheel">
+    <material>Gazebo/Yellow</material>
+  </gazebo>
+  <gazebo reference="right_wheel">
+    <material>Gazebo/Yellow</material>
+  </gazebo>
+  <gazebo reference="camera">
+    <material>Gazebo/Yellow</material>
+  </gazebo>
 </robot>
